File: projects/heavy-lift-uav/kicad/power_and_signal_schematic.kicad_sch (KiCad schematic)
At the start: 0 parts

Commit message: Finalize technical report, calculation walkthroughs, subfolder READMEs, and KiCad/aero assets
Parts:
- added BAT?: 12S LiPo Battery, symbol Connector_Generic:Conn_01x02
- added BMS: BMS Ideal Diode, symbol Connector_Generic:Conn_01x06
- added COMP: Jetson Orin Nano, symbol Connector_Generic:Conn_01x06
- added ESC: Flame120A ESC 1, symbol Connector_Generic:Conn_01x07
- added ESC: Flame120A ESC 6, symbol Connector_Generic:Conn_01x07
- added ESC: Flame120A ESC 2, symbol Connector_Generic:Conn_01x07
- added ESC: Flame120A ESC 4, symbol Connector_Generic:Conn_01x07
- added ESC: Flame120A ESC 5, symbol Connector_Generic:Conn_01x07
- added ESC: Flame120A ESC 3, symbol Connector_Generic:Conn_01x07
- added FC: Pixhawk 6X, symbol Connector_Generic:Conn_01x18
- added GEN: 3.6kW Hybrid Generator, symbol Connector_Generic:Conn_01x04
- added GPS?: Here3 GPS RTK 1, symbol Connector_Generic:Conn_01x04
- added GPS?: Here3 GPS RTK 2, symbol Connector_Generic:Conn_01x04
- added J_PAYLOAD?: 12V Payload, symbol Connector_Generic:Conn_01x02
- added M: T-Motor U15 II 1, symbol Connector_Generic:Conn_01x03
- added M: T-Motor U15 II 4, symbol Connector_Generic:Conn_01x03
- added M: T-Motor U15 II 3, symbol Connector_Generic:Conn_01x03
- added M: T-Motor U15 II 6, symbol Connector_Generic:Conn_01x03
- added M: T-Motor U15 II 2, symbol Connector_Generic:Conn_01x03
- added M: T-Motor U15 II 5, symbol Connector_Generic:Conn_01x03
- added PDB: Power Distribution Board, symbol Connector_Generic:Conn_01x16
- added REG?: DC-DC 5V 10A, symbol Connector_Generic:Conn_01x04
- added REG?: DC-DC 12V 10A, symbol Connector_Generic:Conn_01x04
- added TEL?: RFD900 Telemetry, symbol Connector_Generic:Conn_01x04
Connections:
- new net 48V_BUS: BMS.1 (Pin_1), GEN.1 (Pin_1), PDB.1 (Pin_1)
- new net AUX_V+: PDB.15 (Pin_15), REG?.1 (Pin_1), REG?.1 (Pin_1)
- new net AUX_V-: PDB.16 (Pin_16), REG?.2 (Pin_2), REG?.2 (Pin_2)
- new net BAT_V+: BAT?.1 (Pin_1), BMS.3 (Pin_3)
- new net BAT_V-: BAT?.2 (Pin_2), BMS.4 (Pin_4)
- new net CAN_H: BMS.5 (Pin_5), FC.3 (Pin_3), GEN.3 (Pin_3), GPS?.3 (Pin_3)
- new net CAN_L: BMS.6 (Pin_6), FC.4 (Pin_4), GEN.4 (Pin_4), GPS?.4 (Pin_4)
- new net ESC1_V+: ESC.1 (Pin_1), PDB.3 (Pin_3)
- new net ESC1_V-: ESC.2 (Pin_2), PDB.4 (Pin_4)
- new net ESC2_V+: ESC.1 (Pin_1), PDB.5 (Pin_5)
- new net ESC2_V-: ESC.2 (Pin_2), PDB.6 (Pin_6)
- new net ESC3_V+: ESC.1 (Pin_1), PDB.7 (Pin_7)
- new net ESC3_V-: ESC.2 (Pin_2), PDB.8 (Pin_8)
- new net ESC4_V+: ESC.1 (Pin_1), PDB.9 (Pin_9)
- new net ESC4_V-: ESC.2 (Pin_2), PDB.10 (Pin_10)
- new net ESC5_V+: ESC.1 (Pin_1), PDB.11 (Pin_11)
- new net ESC5_V-: ESC.2 (Pin_2), PDB.12 (Pin_12)
- new net ESC6_V+: ESC.1 (Pin_1), PDB.13 (Pin_13)
- new net ESC6_V-: ESC.2 (Pin_2), PDB.14 (Pin_14)
- new net ETH_RX_N: COMP.4 (Pin_4), FC.18 (Pin_18)
- new net ETH_RX_P: COMP.3 (Pin_3), FC.17 (Pin_17)
- new net ETH_TX_N: COMP.6 (Pin_6), FC.16 (Pin_16)
- new net ETH_TX_P: COMP.5 (Pin_5), FC.15 (Pin_15)
- new net GND_12V: J_PAYLOAD?.1 (Pin_1), REG?.4 (Pin_4)
- new net GND_5V: COMP.2 (Pin_2), FC.2 (Pin_2), GPS?.2 (Pin_2), GPS?.2 (Pin_2), REG?.4 (Pin_4), TEL?.2 (Pin_2)
- new net GND_BUS: BMS.2 (Pin_2), GEN.2 (Pin_2), PDB.2 (Pin_2)
- new net GPS_RXD: FC.6 (Pin_6), GPS?.3 (Pin_3)
- new net GPS_TXD: FC.5 (Pin_5), GPS?.4 (Pin_4)
- new net M1_A: ESC.5 (Pin_5), M.1 (Pin_1)
- new net M1_B: ESC.6 (Pin_6), M.2 (Pin_2)
- new net M1_C: ESC.7 (Pin_7), M.3 (Pin_3)
- new net M2_A: ESC.5 (Pin_5), M.1 (Pin_1)
- new net M2_B: ESC.6 (Pin_6), M.2 (Pin_2)
- new net M2_C: ESC.7 (Pin_7), M.3 (Pin_3)
- new net M3_A: ESC.5 (Pin_5), M.1 (Pin_1)
- new net M3_B: ESC.6 (Pin_6), M.2 (Pin_2)
- new net M3_C: ESC.7 (Pin_7), M.3 (Pin_3)
- new net M4_A: ESC.5 (Pin_5), M.1 (Pin_1)
- new net M4_B: ESC.6 (Pin_6), M.2 (Pin_2)
- new net M4_C: ESC.7 (Pin_7), M.3 (Pin_3)
- new net M5_A: ESC.5 (Pin_5), M.1 (Pin_1)
- new net M5_B: ESC.6 (Pin_6), M.2 (Pin_2)
- new net M5_C: ESC.7 (Pin_7), M.3 (Pin_3)
- new net M6_A: ESC.5 (Pin_5), M.1 (Pin_1)
- new net M6_B: ESC.6 (Pin_6), M.2 (Pin_2)
- new net M6_C: ESC.7 (Pin_7), M.3 (Pin_3)
- new net PWM_1: ESC.3 (Pin_3), FC.9 (Pin_9)
- new net PWM_2: ESC.3 (Pin_3), FC.10 (Pin_10)
- new net PWM_3: ESC.3 (Pin_3), FC.11 (Pin_11)
- new net PWM_4: ESC.3 (Pin_3), FC.12 (Pin_12)
- new net PWM_5: ESC.3 (Pin_3), FC.13 (Pin_13)
- new net PWM_6: ESC.3 (Pin_3), FC.14 (Pin_14)
- new net TEL_RXD: FC.8 (Pin_8), TEL?.3 (Pin_3)
- new net TEL_TXD: FC.7 (Pin_7), TEL?.4 (Pin_4)
- new net VCC_12V: J_PAYLOAD?.2 (Pin_2), REG?.3 (Pin_3)
- new net VCC_5V: COMP.1 (Pin_1), FC.1 (Pin_1), GPS?.1 (Pin_1), GPS?.1 (Pin_1), REG?.3 (Pin_3), TEL?.1 (Pin_1)
- no-connect marks 0 -> 6
Other:
- note added: "BUFFER BATTERY & BMS FAILSAFE Battery: 12S LiPo (44.4V - 50.4V, 4500mAh 45C) Failsafe BMS Parallel Coupling (Ideal Diode)"
- note added: "COMPANION COMPUTER[Nvidia Jetson orin ]"
- note added: "FLIGHT CONTROLLER (Pixhawk 6X) - PWM Outputs [PWM_1 to PWM_6]: 6x ESC Signal Inputs - Telemetry 1: 915 MHz RF Telemetry Radio (1W Output) - GPS / RTK: Dual Neo-3 GPS/RTK Receivers (Serial GPS1 + CAN GPS2) - CAN Bus: Hybrid Generator ECU Telemetry, BMS, and GPS2 - Companion Computer : Ethernet MAVLink to Nvidia Jetson Orin Nano"
- note added: "HYBRID GENERATOR & RECTIFIER SYSTEM Output: 3.6 kW Continuous (48V DC, 75A Max) Fuel: Gasoline 2-Stroke Gen Cable Rating: 48V_BUS, MAX 75A"
- note added: "MAIN POWER DISTRIBUTION BOARD (PDB) Input: 48V DC Bus (Total Hover Power: 3,460.1 W @ 72.1A Total) 6x ESC Branch Outputs: 48V DC, 12.02A Hover"
- note added: "REGULATED RAIL OUTPUTS REG1: 12V 10A Rail for Video Tx / Camera Gimbal REG2: 5V 10A Rail for Flight Controller & Jetson Orin"
- note added: "UAV MAIN POWER PATH (48V HYBRID DC BUS)"
- note removed: "1. FLIGHT CONTROLLER (Pixhawk 6X) - PWM Outputs [PWM_1 .. PWM_6] -> 6x ESC Signal Inputs - Telemetry 1 -> 915 MHz RF Telemetry Radio (1W Output) - GPS / RTK -> Dual Neo-3 GPS/RTK Receivers - CAN Bus [CAN1_H/L] -> Hybrid Generator ECU Telemetry & BMS Status - Companion Computer -> Ethernet MAVLink to Nvidia Jetson Orin Nano"
- note removed: "1. HYBRID GENERATOR & RECTIFIER SYSTEM - Output: 3.6 kW Continuous (48V DC, 75A Max) - Fuel: Gasoline 2-Stroke Gen - Cable Rating: 48V_BUS, MAX 75A"
- note removed: "2. BUFFER BATTERY & BMS FAILSAFE - Battery: 12S LiPo (44.4V - 50.4V, 4500mAh 45C) - Failsafe BMS Parallel Coupling (Ideal Diode) - Cable Rating: BAT_BUS, MAX 100A PEAK"
- note removed: "2. PAYLOAD & VIDEO DOWNLINK - Camera / Gimbal -> 12V Regulated Auxiliary Power Rail (12V, 10A Max) - FPV Video Transmitter -> 5.8GHz VTX Downlink"
- note removed: "3. MAIN POWER DISTRIBUTION BOARD (PDB) - Input: 48V DC Bus (Total Hover Power: 3,460.1 W @ 72.1A Total) - 6x ESC Branch Outputs: 48V DC, 12.02A Hover / 60A Peak per Branch"
- note removed: "HEAVY-LIFT UAV MAIN POWER PATH (48V HYBRID DC BUS)"
- note removed: "WIRE LABEL: [ESC_1_PWR] -> 48V, 12.02A Hover / 60A Peak (120A ESC Rating)"
- note removed: "WIRE LABEL: [ESC_2_PWR] -> 48V, 12.02A Hover / 60A Peak (120A ESC Rating)"
- note removed: "WIRE LABEL: [ESC_3_PWR] -> 48V, 12.02A Hover / 60A Peak (120A ESC Rating)"
- note removed: "WIRE LABEL: [ESC_4_PWR] -> 48V, 12.02A Hover / 60A Peak (120A ESC Rating)"
- note removed: "WIRE LABEL: [ESC_5_PWR] -> 48V, 12.02A Hover / 60A Peak (120A ESC Rating)"
- note removed: "WIRE LABEL: [ESC_6_PWR] -> 48V, 12.02A Hover / 60A Peak (120A ESC Rating)"
- company: Flight Systems Division -> Vaibhav Parashari
- title: Heavy-Lift Gas-Electric Hybrid Hexacopter - Power & Signal Schematic -> Hexacopter - Power & Signal Schematic

Commit message: docs: update UAV design report with 520 Wh/kg battery specific energy, indigenous avionics, and validated CAD/mesh geometries
Parts:
- removed BAT?: 12S LiPo Battery, symbol Connector_Generic:Conn_01x02
- removed BMS: BMS Ideal Diode, symbol Connector_Generic:Conn_01x06
- removed COMP: Jetson Orin Nano, symbol Connector_Generic:Conn_01x06
- removed ESC: Flame120A ESC 1, symbol Connector_Generic:Conn_01x07
- removed ESC: Flame120A ESC 6, symbol Connector_Generic:Conn_01x07
- removed ESC: Flame120A ESC 2, symbol Connector_Generic:Conn_01x07
- removed ESC: Flame120A ESC 4, symbol Connector_Generic:Conn_01x07
- removed ESC: Flame120A ESC 5, symbol Connector_Generic:Conn_01x07
- removed ESC: Flame120A ESC 3, symbol Connector_Generic:Conn_01x07
- removed FC: Pixhawk 6X, symbol Connector_Generic:Conn_01x18
- removed GEN: 3.6kW Hybrid Generator, symbol Connector_Generic:Conn_01x04
- removed GPS?: Here3 GPS RTK 1, symbol Connector_Generic:Conn_01x04
- removed GPS?: Here3 GPS RTK 2, symbol Connector_Generic:Conn_01x04
- removed J_PAYLOAD?: 12V Payload, symbol Connector_Generic:Conn_01x02
- removed M: T-Motor U15 II 1, symbol Connector_Generic:Conn_01x03
- removed M: T-Motor U15 II 4, symbol Connector_Generic:Conn_01x03
- removed M: T-Motor U15 II 3, symbol Connector_Generic:Conn_01x03
- removed M: T-Motor U15 II 6, symbol Connector_Generic:Conn_01x03
- removed M: T-Motor U15 II 2, symbol Connector_Generic:Conn_01x03
- removed M: T-Motor U15 II 5, symbol Connector_Generic:Conn_01x03
- removed PDB: Power Distribution Board, symbol Connector_Generic:Conn_01x16
- removed REG?: DC-DC 5V 10A, symbol Connector_Generic:Conn_01x04
- removed REG?: DC-DC 12V 10A, symbol Connector_Generic:Conn_01x04
- removed TEL?: RFD900 Telemetry, symbol Connector_Generic:Conn_01x04
- added BAT1: 12S 520Wh/kg SSS Battery, symbol Connector_Generic:Conn_01x02
- added BMS1: BMS & Protection, symbol Connector_Generic:Conn_01x06
- added COMP1: Jetson Orin Nano, symbol Connector_Generic:Conn_01x06
- added ESC1: Flame120A ESC 1, symbol Connector_Generic:Conn_01x07
- added ESC2: Flame120A ESC 2, symbol Connector_Generic:Conn_01x07
- added ESC3: Flame120A ESC 3, symbol Connector_Generic:Conn_01x07
- added ESC4: Flame120A ESC 4, symbol Connector_Generic:Conn_01x07
- added ESC5: Flame120A ESC 5, symbol Connector_Generic:Conn_01x07
- added ESC6: Flame120A ESC 6, symbol Connector_Generic:Conn_01x07
- added FC1: BRAHMA F7 Autopilot, symbol Connector_Generic:Conn_01x18
- added GEN1: External Charger Port, symbol Connector_Generic:Conn_01x04
- added GPS1: Elena Geo NDNU GPS, symbol Connector_Generic:Conn_01x04
- added GPS2: Secondary GPS, symbol Connector_Generic:Conn_01x04
- added J_PAYLOAD: 12V Payload, symbol Connector_Generic:Conn_01x02
- added M1: T-Motor U15 II 1, symbol Connector_Generic:Conn_01x03
- added M2: T-Motor U15 II 2, symbol Connector_Generic:Conn_01x03
- added M3: T-Motor U15 II 3, symbol Connector_Generic:Conn_01x03
- added M4: T-Motor U15 II 4, symbol Connector_Generic:Conn_01x03
- added M5: T-Motor U15 II 5, symbol Connector_Generic:Conn_01x03
- added M6: T-Motor U15 II 6, symbol Connector_Generic:Conn_01x03
- added PDB1: Power Distribution Board, symbol Connector_Generic:Conn_01x16
- added REG1: DC-DC 12V 10A, symbol Connector_Generic:Conn_01x04
- added REG2: DC-DC 5V 10A, symbol Connector_Generic:Conn_01x04
- added TEL1: ZeroDrag Nexus1 ELRS, symbol Connector_Generic:Conn_01x04
Connections:
- net 48V_BUS: now also BMS1.1 (Pin_1), GEN1.1 (Pin_1), PDB1.1 (Pin_1)
- net AUX_V+: now also PDB1.15 (Pin_15), REG1.1 (Pin_1), REG2.1 (Pin_1)
- net AUX_V-: now also PDB1.16 (Pin_16), REG1.2 (Pin_2), REG2.2 (Pin_2)
- net BAT_V+: now also BAT1.1 (Pin_1), BMS1.3 (Pin_3)
- net BAT_V-: now also BAT1.2 (Pin_2), BMS1.4 (Pin_4)
- net CAN_H: now also BMS1.5 (Pin_5), FC1.3 (Pin_3), GEN1.3 (Pin_3), GPS2.3 (Pin_3)
- net CAN_L: now also BMS1.6 (Pin_6), FC1.4 (Pin_4), GEN1.4 (Pin_4), GPS2.4 (Pin_4)
- net ESC1_V+: now also ESC1.1 (Pin_1), PDB1.3 (Pin_3)
- net ESC1_V-: now also ESC1.2 (Pin_2), PDB1.4 (Pin_4)
- net ESC2_V+: now also ESC2.1 (Pin_1), PDB1.5 (Pin_5)
- net ESC2_V-: now also ESC2.2 (Pin_2), PDB1.6 (Pin_6)
- net ESC3_V+: now also ESC3.1 (Pin_1), PDB1.7 (Pin_7)
- net ESC3_V-: now also ESC3.2 (Pin_2), PDB1.8 (Pin_8)
- net ESC4_V+: now also ESC4.1 (Pin_1), PDB1.9 (Pin_9)
- net ESC4_V-: now also ESC4.2 (Pin_2), PDB1.10 (Pin_10)
- net ESC5_V+: now also ESC5.1 (Pin_1), PDB1.11 (Pin_11)
- net ESC5_V-: now also ESC5.2 (Pin_2), PDB1.12 (Pin_12)
- net ESC6_V+: now also ESC6.1 (Pin_1), PDB1.13 (Pin_13)
- net ESC6_V-: now also ESC6.2 (Pin_2), PDB1.14 (Pin_14)
- net ETH_RX_N: now also COMP1.4 (Pin_4), FC1.18 (Pin_18)
- net ETH_RX_P: now also COMP1.3 (Pin_3), FC1.17 (Pin_17)
- net ETH_TX_N: now also COMP1.6 (Pin_6), FC1.16 (Pin_16)
- net ETH_TX_P: now also COMP1.5 (Pin_5), FC1.15 (Pin_15)
- net GND_12V: now also J_PAYLOAD.1 (Pin_1), REG1.4 (Pin_4)
- net GND_5V: now also COMP1.2 (Pin_2), FC1.2 (Pin_2), GPS1.2 (Pin_2), GPS2.2 (Pin_2), REG2.4 (Pin_4), TEL1.2 (Pin_2)
- net GND_BUS: now also BMS1.2 (Pin_2), GEN1.2 (Pin_2), PDB1.2 (Pin_2)
- net GPS_RXD: now also FC1.6 (Pin_6), GPS1.3 (Pin_3)
- net GPS_TXD: now also FC1.5 (Pin_5), GPS1.4 (Pin_4)
- net M1_A: now also ESC1.5 (Pin_5), M1.1 (Pin_1)
- net M1_B: now also ESC1.6 (Pin_6), M1.2 (Pin_2)
- net M1_C: now also ESC1.7 (Pin_7), M1.3 (Pin_3)
- net M2_A: now also ESC2.5 (Pin_5), M2.1 (Pin_1)
- net M2_B: now also ESC2.6 (Pin_6), M2.2 (Pin_2)
- net M2_C: now also ESC2.7 (Pin_7), M2.3 (Pin_3)
- net M3_A: now also ESC3.5 (Pin_5), M3.1 (Pin_1)
- net M3_B: now also ESC3.6 (Pin_6), M3.2 (Pin_2)
- net M3_C: now also ESC3.7 (Pin_7), M3.3 (Pin_3)
- net M4_A: now also ESC4.5 (Pin_5), M4.1 (Pin_1)
- net M4_B: now also ESC4.6 (Pin_6), M4.2 (Pin_2)
- net M4_C: now also ESC4.7 (Pin_7), M4.3 (Pin_3)
- net M5_A: now also ESC5.5 (Pin_5), M5.1 (Pin_1)
- net M5_B: now also ESC5.6 (Pin_6), M5.2 (Pin_2)
- net M5_C: now also ESC5.7 (Pin_7), M5.3 (Pin_3)
- net M6_A: now also ESC6.5 (Pin_5), M6.1 (Pin_1)
- net M6_B: now also ESC6.6 (Pin_6), M6.2 (Pin_2)
- net M6_C: now also ESC6.7 (Pin_7), M6.3 (Pin_3)
- net PWM_1: now also ESC1.3 (Pin_3), FC1.9 (Pin_9)
- net PWM_2: now also ESC2.3 (Pin_3), FC1.10 (Pin_10)
- net PWM_3: now also ESC3.3 (Pin_3), FC1.11 (Pin_11)
- net PWM_4: now also ESC4.3 (Pin_3), FC1.12 (Pin_12)
- net PWM_5: now also ESC5.3 (Pin_3), FC1.13 (Pin_13)
- net PWM_6: now also ESC6.3 (Pin_3), FC1.14 (Pin_14)
- net TEL_RXD: now also FC1.8 (Pin_8), TEL1.3 (Pin_3)
- net TEL_TXD: now also FC1.7 (Pin_7), TEL1.4 (Pin_4)
- net VCC_12V: now also J_PAYLOAD.2 (Pin_2), REG1.3 (Pin_3)
- net VCC_5V: now also COMP1.1 (Pin_1), FC1.1 (Pin_1), GPS1.1 (Pin_1), GPS2.1 (Pin_1), REG2.3 (Pin_3), TEL1.1 (Pin_1)
Other:
- note added: "1. BATTERY CHARGER SYSTEM - Output: Ground Balance Charger Port - Cable Rating: 48V_BUS, MAX 10A (Ground Charging Only)"
- note added: "1. FLIGHT CONTROLLER (Darkmatter BRAHMA F7) - PWM Outputs [PWM_1 .. PWM_6] -> 6x ESC Signal Inputs - Telemetry 1 -> ZeroDrag Nexus1 ELRS Link (2.4GHz) - GPS / RTK -> Elena Geo NDNU GPS/RTK Receiver (Serial GPS1) - CAN Bus [CAN1_H/L] -> BMS Telemetry, and GPS2 - Companion Computer -> Ethernet MAVLink to Nvidia Jetson Orin Nano"
- note added: "2. COMPANION COMPUTER - Model: Nvidia Jetson Orin Nano - High-level autonomy and payload interface - Powered by DC-DC 5V Regulator"
- note added: "2. MAIN PROPULSION BATTERY & BMS - Battery: 12S Semi-Solid-State (44.4V Nominal, 520 Wh/kg) - Pack Capacity: 6,307.2 Wh (12.129 kg Pack Mass) - Cable Rating: BAT_BUS, MAX 100A continuous / 150A Peak"
- note added: "3. MAIN POWER DISTRIBUTION BOARD (PDB) - Input: 48V DC Bus (Total Hover Power: 3,836.1 W @ 86.3A Total) - 6x ESC Branch Outputs: 48V DC, 14.4A Hover / 53.0A Peak per Branch"
- note added: "3. REGULATED RAIL OUTPUTS - REG1: 12V 10A Rail for Video Tx / Camera Gimbal - REG2: 5V 10A Rail for Flight Controller & Jetson Orin"
- note added: "HEAVY-LIFT UAV MAIN POWER PATH (48V BATTERY-ELECTRIC DC BUS)"
- note removed: "BUFFER BATTERY & BMS FAILSAFE Battery: 12S LiPo (44.4V - 50.4V, 4500mAh 45C) Failsafe BMS Parallel Coupling (Ideal Diode)"
- note removed: "COMPANION COMPUTER[Nvidia Jetson orin ]"
- note removed: "FLIGHT CONTROLLER (Pixhawk 6X) - PWM Outputs [PWM_1 to PWM_6]: 6x ESC Signal Inputs - Telemetry 1: 915 MHz RF Telemetry Radio (1W Output) - GPS / RTK: Dual Neo-3 GPS/RTK Receivers (Serial GPS1 + CAN GPS2) - CAN Bus: Hybrid Generator ECU Telemetry, BMS, and GPS2 - Companion Computer : Ethernet MAVLink to Nvidia Jetson Orin Nano"
- note removed: "HYBRID GENERATOR & RECTIFIER SYSTEM Output: 3.6 kW Continuous (48V DC, 75A Max) Fuel: Gasoline 2-Stroke Gen Cable Rating: 48V_BUS, MAX 75A"
- note removed: "MAIN POWER DISTRIBUTION BOARD (PDB) Input: 48V DC Bus (Total Hover Power: 3,460.1 W @ 72.1A Total) 6x ESC Branch Outputs: 48V DC, 12.02A Hover"
- note removed: "REGULATED RAIL OUTPUTS REG1: 12V 10A Rail for Video Tx / Camera Gimbal REG2: 5V 10A Rail for Flight Controller & Jetson Orin"
- note removed: "UAV MAIN POWER PATH (48V HYBRID DC BUS)"
- company: Vaibhav Parashari -> Flight Systems Division
- title: Hexacopter - Power & Signal Schematic -> Heavy-Lift Battery-Electric Hexacopter - Power & Signal Schematic
